File: R2-mechanisms.sch (EAGLE design)
At the start: 22 parts, among them IC1 ULN2003AN

Commit message: Update
Connections:
- net 12V: now also C1G$1.KL, C2G$1.KL, C3G$1.KL
- net GND: no longer C1G$1.KL, C2G$1.KL, C3G$1.KL
Changed lines of the file:
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@@
 <setting verticaltext="up"/>
 </settings>
-<grid distance="0.1" unitdist="inch" unit="mm" style="lines" multiple="1" display="yes" altdistance="0.01" altunitdist="inch" altunit="mm"/>
+<grid distance="0.1" unitdist="inch" unit="inch" style="lines" multiple="1" display="no" altdistance="0.01" altunitdist="inch" altunit="inch"/>
 <layers>
 <layer number="1" name="Top" color="4" fill="1" visible="no" active="no"/>
@@
 </segment>
 <segment>
+<pinref part="IC1" gate="A" pin="GND"/>
+<wire x1="86.36" y1="127" x2="81.28" y2="127" width="0.1524" layer="91" grouprefs="MECHANISMS"/>
+<label x="83.82" y="127" size="1.27" layer="95" rot="R180" xref="yes" grouprefs="MECHANISMS"/>
+</segment>
+<segment>
+<pinref part="JP5" gate="G$1" pin="2"/>
+<wire x1="116.84" y1="182.88" x2="111.76" y2="182.88" width="0.1524" layer="91" grouprefs="SWTCHES"/>
+<label x="111.76" y="182.88" size="1.27" layer="95" rot="R180" xref="yes" grouprefs="SWTCHES"/>
+</segment>
+<segment>
+<pinref part="JP6" gate="G$1" pin="2"/>
+<wire x1="88.9" y1="182.88" x2="83.82" y2="182.88" width="0.1524" layer="91" grouprefs="SWTCHES"/>
+<label x="83.82" y="182.88" size="1.27" layer="95" rot="R180" xref="yes" grouprefs="SWTCHES"/>
+</segment>
+<segment>
+<pinref part="JP7" gate="G$1" pin="2"/>
+<wire x1="60.96" y1="182.88" x2="55.88" y2="182.88" width="0.1524" layer="91" grouprefs="SWTCHES"/>
+<label x="55.88" y="182.88" size="1.27" layer="95" rot="R180" xref="yes" grouprefs="SWTCHES"/>
+</segment>
+<segment>
+<pinref part="IN" gate="G$2" pin="KL"/>
+<wire x1="15.24" y1="104.14" x2="20.32" y2="104.14" width="0.1524" layer="91" grouprefs="POWER"/>
+<label x="20.32" y="104.14" size="1.27" layer="95" xref="yes" grouprefs="POWER"/>
+</segment>
+<segment>
+<pinref part="ENC1" gate="G$1" pin="GND"/>
+<wire x1="147.32" y1="147.32" x2="144.78" y2="147.32" width="0.1524" layer="91" grouprefs="ENCODER"/>
+<label x="144.78" y="147.32" size="1.27" layer="95" rot="R180" xref="yes" grouprefs="ENCODER"/>
+</segment>
+</net>
+<net name="12V" class="0">
+<segment>
+<pinref part="IC1" gate="A" pin="CD+"/>
+<wire x1="111.76" y1="127" x2="116.84" y2="127" width="0.1524" layer="91" grouprefs="MECHANISMS"/>
+<label x="116.84" y="127" size="1.27" layer="95" xref="yes" grouprefs="MECHANISMS"/>
+</segment>
+<segment>
+<pinref part="IN" gate="G$1" pin="KL"/>
+<wire x1="15.24" y1="109.22" x2="20.32" y2="109.22" width="0.1524" layer="91" grouprefs="POWER"/>
+<label x="20.32" y="109.22" size="1.27" layer="95" xref="yes" grouprefs="POWER"/>
+</segment>
+<segment>
+<pinref part="C1" gate="G$1" pin="KL"/>
+<wire x1="53.34" y1="149.86" x2="58.42" y2="149.86" width="0.1524" layer="91" grouprefs="MECHANISMS"/>
+<label x="58.42" y="149.86" size="1.27" layer="95" xref="yes" grouprefs="MECHANISMS"/>
+</segment>
+<segment>
+<pinref part="C2" gate="G$1" pin="KL"/>
+<wire x1="53.34" y1="139.7" x2="58.42" y2="139.7" width="0.1524" layer="91" grouprefs="MECHANISMS"/>
+<label x="58.42" y="139.7" size="1.27" layer="95" xref="yes" grouprefs="MECHANISMS"/>
+</segment>
+<segment>
 <pinref part="C3" gate="G$1" pin="KL"/>
 <wire x1="53.34" y1="129.54" x2="58.42" y2="129.54" width="0.1524" layer="91" grouprefs="MECHANISMS"/>
 <label x="58.42" y="129.54" size="1.27" layer="95" xref="yes" grouprefs="MECHANISMS"/>
 </segment>
-<segment>
-<pinref part="C2" gate="G$1" pin="KL"/>
-<wire x1="53.34" y1="139.7" x2="58.42" y2="139.7" width="0.1524" layer="91" grouprefs="MECHANISMS"/>
-<label x="58.42" y="139.7" size="1.27" layer="95" xref="yes" grouprefs="MECHANISMS"/>
-</segment>
-<segment>
-<pinref part="C1" gate="G$1" pin="KL"/>
-<wire x1="53.34" y1="149.86" x2="58.42" y2="149.86" width="0.1524" layer="91" grouprefs="MECHANISMS"/>
-<label x="58.42" y="149.86" size="1.27" layer="95" xref="yes" grouprefs="MECHANISMS"/>
-</segment>
-<segment>
-<pinref part="IC1" gate="A" pin="GND"/>
-<wire x1="86.36" y1="127" x2="81.28" y2="127" width="0.1524" layer="91" grouprefs="MECHANISMS"/>
-<label x="83.82" y="127" size="1.27" layer="95" rot="R180" xref="yes" grouprefs="MECHANISMS"/>
-</segment>
-<segment>
-<pinref part="JP5" gate="G$1" pin="2"/>
-<wire x1="116.84" y1="182.88" x2="111.76" y2="182.88" width="0.1524" layer="91" grouprefs="SWTCHES"/>
-<label x="111.76" y="182.88" size="1.27" layer="95" rot="R180" xref="yes" grouprefs="SWTCHES"/>
-</segment>
-<segment>
-<pinref part="JP6" gate="G$1" pin="2"/>
-<wire x1="88.9" y1="182.88" x2="83.82" y2="182.88" width="0.1524" layer="91" grouprefs="SWTCHES"/>
-<label x="83.82" y="182.88" size="1.27" layer="95" rot="R180" xref="yes" grouprefs="SWTCHES"/>
-</segment>
-<segment>
-<pinref part="JP7" gate="G$1" pin="2"/>
-<wire x1="60.96" y1="182.88" x2="55.88" y2="182.88" width="0.1524" layer="91" grouprefs="SWTCHES"/>
-<label x="55.88" y="182.88" size="1.27" layer="95" rot="R180" xref="yes" grouprefs="SWTCHES"/>
-</segment>
-<segment>
-<pinref part="IN" gate="G$2" pin="KL"/>
-<wire x1="15.24" y1="104.14" x2="20.32" y2="104.14" width="0.1524" layer="91" grouprefs="POWER"/>
-<label x="20.32" y="104.14" size="1.27" layer="95" xref="yes" grouprefs="POWER"/>
-</segment>
-<segment>
-<pinref part="ENC1" gate="G$1" pin="GND"/>
-<wire x1="147.32" y1="147.32" x2="144.78" y2="147.32" width="0.1524" layer="91" grouprefs="ENCODER"/>
-<label x="144.78" y="147.32" size="1.27" layer="95" rot="R180" xref="yes" grouprefs="ENCODER"/>
-</segment>
-</net>
-<net name="12V" class="0">
-<segment>
-<pinref part="IC1" gate="A" pin="CD+"/>
-<wire x1="111.76" y1="127" x2="116.84" y2="127" width="0.1524" layer="91" grouprefs="MECHANISMS"/>
-<label x="116.84" y="127" size="1.27" layer="95" xref="yes" grouprefs="MECHANISMS"/>
-</segment>
-<segment>
-<pinref part="IN" gate="G$1" pin="KL"/>
-<wire x1="15.24" y1="109.22" x2="20.32" y2="109.22" width="0.1524" layer="91" grouprefs="POWER"/>
-<label x="20.32" y="109.22" size="1.27" layer="95" xref="yes" grouprefs="POWER"/>
-</segment>
-</net>
+</net>
