File: R2-mechanisms.brd (EAGLE design)
At the start: 70.8 x 80 mm, 22 parts, among them IC1 ULN2003AN

Commit message: Update
Connections:
- net 12V: now also C1.1, C2.1, C3.1
- net GND: no longer C1.1, C2.1, C3.1
Routing:
- net GND: track 414.6 -> 327.2 mm
- net 12V: track 10.5 -> 81.2 mm
Changed lines of the file:
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@@
 <contactref element="ZX1" pad="39"/>
 <contactref element="CYTRON" pad="5"/>
-<contactref element="C3" pad="1"/>
-<contactref element="C2" pad="1"/>
-<contactref element="C1" pad="1"/>
 <contactref element="IC1" pad="8"/>
 <contactref element="JP5" pad="2"/>
@@
 <wire x1="5.461" y1="20.5232" x2="14.4272" y2="20.5232" width="1.27" layer="16"/>
 <wire x1="14.4272" y1="20.5232" x2="15.24" y2="21.336" width="1.27" layer="16"/>
-<wire x1="4.699" y1="20.5232" x2="2.286" y2="18.1102" width="1.27" layer="16"/>
 <wire x1="5.461" y1="20.5232" x2="4.699" y2="20.5232" width="1.27" layer="16"/>
-<wire x1="11.43" y1="5.715" x2="11.43" y2="4.4704" width="1.27" layer="16"/>
-<wire x1="11.43" y1="4.4704" x2="11.4046" y2="4.445" width="1.27" layer="16"/>
-<wire x1="24.1046" y1="3.5306" x2="24.1046" y2="4.445" width="1.27" layer="16"/>
-<wire x1="36.83" y1="4.445" x2="36.8046" y2="4.445" width="1.27" layer="16"/>
-<wire x1="11.176" y1="2.921" x2="12.065" y2="2.032" width="1.27" layer="16"/>
-<wire x1="11.4046" y1="4.445" x2="11.176" y2="4.2164" width="1.27" layer="16"/>
-<wire x1="11.176" y1="4.2164" x2="11.176" y2="2.921" width="1.27" layer="16"/>
-<wire x1="2.286" y1="12.954" x2="2.286" y2="18.1102" width="1.27" layer="16"/>
 <wire x1="7.112" y1="72.517" x2="7.112" y2="73.787" width="1.27" layer="16"/>
 <wire x1="7.112" y1="73.787" x2="8.499" y2="75.174" width="1.27" layer="16"/>
@@
 <wire x1="7.62" y1="48.26" x2="6.35" y2="49.53" width="1.27" layer="16"/>
 <wire x1="7.62" y1="48.26" x2="6.35" y2="46.99" width="1.27" layer="16"/>
-<wire x1="40.64309375" y1="2.833871875" x2="45.72285625" y2="2.7804" width="1.016" layer="16"/>
-<wire x1="35.630771875" y1="1.616634375" x2="36.833515625" y2="1.603971875" width="1.016" layer="16"/>
-<wire x1="36.833515625" y1="1.603971875" x2="37.78953125" y2="1.593909375" width="1.016" layer="16"/>
 <wire x1="45.7227875" y1="2.804665625" x2="46.736" y2="2.794" width="1.016" layer="16"/>
 <wire x1="45.7227875" y1="2.804665625" x2="45.721384375" y2="3.31083125" width="1.016" layer="16"/>
@@
 <wire x1="10.16" y1="66.294" x2="10.16" y2="67.564" width="1.27" layer="16"/>
 <contactref element="ENC1" pad="2"/>
-<wire x1="35.709765625" y1="1.628234375" x2="35.687" y2="1.651" width="1.016" layer="16"/>
-<wire x1="36.262" y1="1.616634375" x2="35.698165625" y2="1.616634375" width="1.016" layer="16"/>
 <wire x1="55.88" y1="34.29" x2="55.88" y2="31.75" width="1.016" layer="16"/>
 <wire x1="55.88" y1="31.75" x2="59.182" y2="28.448" width="1.016" layer="16"/>
@@
 <wire x1="67.945" y1="21.59" x2="69.215" y2="20.32" width="1.016" layer="16"/>
 <wire x1="67.945" y1="21.59" x2="69.215" y2="22.86" width="1.016" layer="16"/>
-<wire x1="45.72" y1="5.08" x2="45.72" y2="2.807453125" width="1.016" layer="16"/>
 <wire x1="45.72" y1="2.807453125" x2="45.7227875" y2="2.804665625" width="1.016" layer="16"/>
-<wire x1="12.065" y1="2.032" x2="12.468765625" y2="1.628234375" width="1.016" layer="16"/>
-<wire x1="12.468765625" y1="1.628234375" x2="13.716" y2="1.628234375" width="1.016" layer="16"/>
-<wire x1="13.716" y1="1.628234375" x2="23.876" y2="1.628234375" width="1.016" layer="16"/>
-<wire x1="23.876" y1="1.628234375" x2="24.787765625" y2="1.628234375" width="1.016" layer="16"/>
-<wire x1="35.709765625" y1="1.628234375" x2="35.56" y2="1.628234375" width="1.016" layer="16"/>
-<wire x1="35.56" y1="1.628234375" x2="24.787765625" y2="1.628234375" width="1.016" layer="16"/>
-<wire x1="24.1046" y1="4.445" x2="23.876" y2="4.2164" width="1.016" layer="16"/>
-<wire x1="23.876" y1="4.2164" x2="23.876" y2="2.54" width="1.016" layer="16"/>
-<wire x1="23.876" y1="2.54" x2="23.876" y2="1.628234375" width="1.016" layer="16"/>
-<wire x1="23.876" y1="2.54" x2="24.1046" y2="2.3114" width="1.016" layer="16"/>
-<wire x1="12.065" y1="2.032" x2="11.557" y2="1.524" width="1.016" layer="16"/>
-<wire x1="4.826" y1="1.524" x2="11.176" y2="1.524" width="1.016" layer="16"/>
-<wire x1="11.176" y1="1.524" x2="11.557" y2="1.524" width="1.016" layer="16"/>
-<wire x1="4.826" y1="1.524" x2="2.286" y2="4.064" width="1.016" layer="16"/>
-<wire x1="2.286" y1="4.064" x2="2.286" y2="12.954" width="1.016" layer="16"/>
-<wire x1="11.557" y1="1.524" x2="13.611765625" y2="1.524" width="1.016" layer="16"/>
-<wire x1="13.611765625" y1="1.524" x2="13.716" y2="1.628234375" width="1.016" layer="16"/>
-<wire x1="11.176" y1="2.921" x2="11.176" y2="1.524" width="1.016" layer="16"/>
-<wire x1="36.4906" y1="1.845234375" x2="36.262" y2="1.616634375" width="1.016" layer="16"/>
-<wire x1="35.698165625" y1="1.616634375" x2="35.709765625" y2="1.628234375" width="1.016" layer="16"/>
-<wire x1="36.8046" y1="4.445" x2="36.8046" y2="5.0546" width="1.016" layer="16"/>
-<wire x1="36.8046" y1="5.0546" x2="36.83" y2="5.08" width="1.016" layer="16"/>
-<wire x1="24.787765625" y1="1.628234375" x2="24.1046" y2="2.3114" width="1.016" layer="16"/>
-<wire x1="24.1046" y1="2.3114" x2="24.1046" y2="4.445" width="1.016" layer="16"/>
-<wire x1="37.78953125" y1="1.593909375" x2="39.40313125" y2="1.593909375" width="1.016" layer="16"/>
-<wire x1="39.40313125" y1="1.593909375" x2="40.64309375" y2="2.833871875" width="1.016" layer="16"/>
-<wire x1="36.833515625" y1="1.603971875" x2="36.8046" y2="1.6328875" width="1.016" layer="16"/>
-<wire x1="36.8046" y1="1.6328875" x2="36.8046" y2="2.872834375" width="1.016" layer="16"/>
-<wire x1="36.833515625" y1="1.603971875" x2="37.77946875" y2="1.603971875" width="1.016" layer="16"/>
-<wire x1="37.77946875" y1="1.603971875" x2="37.78953125" y2="1.593909375" width="1.016" layer="16"/>
-<wire x1="35.56" y1="1.628234375" x2="36.8046" y2="2.872834375" width="1.016" layer="16"/>
-<wire x1="36.8046" y1="4.445" x2="36.8046" y2="2.872834375" width="1.016" layer="16"/>
 <wire x1="10.16" y1="66.294" x2="12.7" y2="66.294" width="0" layer="19" extent="1-1"/>
 </signal>
@@
 <wire x1="12.4206" y1="15.5194" x2="14.224" y2="13.716" width="1.27" layer="16"/>
 <wire x1="14.224" y1="13.716" x2="15.24" y2="13.716" width="1.27" layer="16"/>
+<contactref element="C1" pad="1"/>
+<wire x1="11.43" y1="5.715" x2="11.43" y2="4.4704" width="1.27" layer="16"/>
+<wire x1="11.43" y1="4.4704" x2="11.4046" y2="4.445" width="1.27" layer="16"/>
+<contactref element="C2" pad="1"/>
+<wire x1="24.1046" y1="3.5306" x2="24.1046" y2="4.445" width="1.27" layer="16"/>
+<contactref element="C3" pad="1"/>
+<wire x1="36.83" y1="4.445" x2="36.8046" y2="4.445" width="1.27" layer="16"/>
+<wire x1="36.8046" y1="4.445" x2="36.8046" y2="5.0546" width="1.016" layer="16"/>
+<wire x1="36.8046" y1="5.0546" x2="36.83" y2="5.08" width="1.016" layer="16"/>
+<wire x1="5.461" y1="15.5194" x2="4.0894" y2="15.5194" width="1.27" layer="16"/>
+<wire x1="2.54" y1="13.97" x2="2.54" y2="2.54" width="1.27" layer="16"/>
+<wire x1="2.54" y1="2.54" x2="3.429" y2="1.651" width="1.27" layer="16"/>
+<wire x1="3.429" y1="1.651" x2="10.16" y2="1.651" width="1.27" layer="16"/>
+<wire x1="10.16" y1="1.651" x2="11.43" y2="2.921" width="1.27" layer="16"/>
+<wire x1="11.43" y1="4.4196" x2="11.43" y2="4.4704" width="1.27" layer="16"/>
+<wire x1="4.0894" y1="15.5194" x2="2.54" y2="13.97" width="1.27" layer="16"/>
+<wire x1="10.16" y1="1.651" x2="11.43" y2="1.651" width="1.27" layer="16"/>
+<wire x1="11.43" y1="1.651" x2="12.7" y2="1.651" width="1.27" layer="16"/>
+<wire x1="12.7" y1="1.651" x2="22.225" y2="1.651" width="1.27" layer="16"/>
+<wire x1="22.225" y1="1.651" x2="24.1046" y2="3.5306" width="1.27" layer="16"/>
+<wire x1="22.225" y1="1.651" x2="24.13" y2="1.651" width="1.27" layer="16"/>
+<wire x1="24.13" y1="1.651" x2="25.4" y2="1.651" width="1.27" layer="16"/>
+<wire x1="25.4" y1="1.651" x2="35.941" y2="1.651" width="1.27" layer="16"/>
+<wire x1="35.941" y1="1.651" x2="36.83" y2="2.54" width="1.27" layer="16"/>
+<wire x1="36.83" y1="2.54" x2="36.83" y2="5.0292" width="1.27" layer="16"/>
+<wire x1="36.83" y1="5.0292" x2="36.8046" y2="5.0546" width="1.27" layer="16"/>
+<wire x1="11.4046" y1="4.445" x2="11.43" y2="4.4196" width="1.27" layer="16"/>
+<wire x1="11.43" y1="4.4196" x2="11.43" y2="2.921" width="1.27" layer="16"/>
+<wire x1="11.43" y1="2.921" x2="11.43" y2="1.651" width="1.27" layer="16"/>
+<wire x1="24.1046" y1="4.445" x2="24.1046" y2="1.6764" width="1.27" layer="16"/>
+<wire x1="24.1046" y1="1.6764" x2="24.13" y2="1.651" width="1.27" layer="16"/>
+<wire x1="24.1046" y1="4.445" x2="24.1046" y2="2.9464" width="1.27" layer="16"/>
+<wire x1="24.1046" y1="2.9464" x2="25.4" y2="1.651" width="1.27" layer="16"/>
+<wire x1="12.7" y1="1.651" x2="11.43" y2="2.921" width="1.27" layer="16"/>
 </signal>
 <signal name="O1">

Commit message: Update
Routing:
- net O1: track 49.2 -> 49.9 mm
Changed lines of the file:
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@@
 <wire x1="17.78" y1="9.525" x2="17.78" y2="8.255" width="1.27" layer="16"/>
 <wire x1="19.05" y1="8.255" x2="19.05" y2="6.985" width="1.27" layer="16"/>
-<wire x1="19.05" y1="6.985" x2="19.05" y2="3.175" width="1.27" layer="16"/>
+<wire x1="19.05" y1="6.985" x2="19.05" y2="3.81" width="1.27" layer="16"/>
+<wire x1="19.05" y1="3.81" x2="19.05" y2="3.175" width="1.27" layer="16"/>
 <wire x1="31.8008" y1="4.445" x2="31.75" y2="4.4958" width="1.27" layer="16"/>
 <wire x1="31.75" y1="4.4958" x2="31.75" y2="5.715" width="1.27" layer="16"/>
@@
 <wire x1="6.4008" y1="4.445" x2="6.4008" y2="3.8608" width="1.016" layer="16"/>
 <wire x1="6.4008" y1="3.8608" x2="6.35" y2="3.81" width="1.016" layer="16"/>
-<wire x1="19.05" y1="3.175" x2="19.1008" y2="4.445" width="0" layer="19" extent="16-16"/>
+<wire x1="19.1008" y1="4.445" x2="19.1008" y2="3.8608" width="1.27" layer="16"/>
+<wire x1="19.1008" y1="3.8608" x2="19.05" y2="3.81" width="1.27" layer="16"/>
 </signal>
 <signal name="N$8">
@@
 <mfgpreviewcolor name="substratecolor" color="0xFF786E46"/>
 </mfgpreviewcolors>
+<errors>
+</errors>
 </board>
 </drawing>
